File: PCBschematic/untitled.kicad_sch (KiCad schematic)
At the start: 4 parts, among them J3 Conn_01x02, Q1 SQ2310ES

Commit message: schematicavancee
Parts:
- added U3: NCS210, Package_TO_SOT_SMD:SOT-363_SC-70-6, symbol Amplifier_Current:NCS210
Connections:
- net GND: now also U3.2 (GND)
- net VCC: now also U3.4 (+IN)
- net at D2.1 (K), J3.1 (Pin_1), R1.2: now also U3.5 (-IN)
Changed lines of the file:
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@@
   (junction (at 68.58 59.69) (diameter 0) (color 0 0 0 0)
   )
-  (wire (pts (xy 68.58 54.61) (xy 86.36 54.61))
+  (wire (pts (xy 68.58 54.61) (xy 91.44 54.61))
     (stroke (width 0) (type default))
   )
@@
     (stroke (width 0) (type default))
   )
+  (wire (pts (xy 101.6 64.77) (xy 101.6 66.04))
+    (stroke (width 0) (type default))
+  )
   (wire (pts (xy 57.15 78.74) (xy 60.96 78.74))
     (stroke (width 0) (type default))
@@
     (stroke (width 0) (type default))
   )
-  (wire (pts (xy 86.36 59.69) (xy 68.58 59.69))
+  (wire (pts (xy 68.58 59.69) (xy 91.44 59.69))
     (stroke (width 0) (type default))
   )
@@
   )
   (text "4 Moteurs\n" (at 35.56 38.1 0)
-    (effects (font (size 1.27 1.27)) (justify left bottom))
+    (effects (font (size 2 2) (thickness 0.4) bold) (justify left bottom))
   )
   (global_label "PWM_1" (shape input) (at 57.15 78.74 180) (fields_autoplaced)
@@
     )
   )
-  (symbol (lib_id "power:GND") (at 91.44 64.77 0) (unit 1)
+  (symbol (lib_id "Amplifier_Current:NCS210") (at 101.6 57.15 0) (unit 1)
     (in_bom yes) (on_board yes) (dnp no) (fields_autoplaced)
-    (property "Reference" "#PWR04" (at 91.44 71.12 0)
+    (property "Reference" "U3" (at 103.5559 45.72 0)
+      (effects (font (size 1.27 1.27)) (justify left))
+    )
+    (property "Value" "NCS210" (at 103.5559 48.26 0)
+      (effects (font (size 1.27 1.27)) (justify left))
+    )
+    (property "Footprint" "Package_TO_SOT_SMD:SOT-363_SC-70-6" (at 101.6 57.15 0)
       (effects (font (size 1.27 1.27)) hide)
     )
-    (property "Value" "GND" (at 91.44 69.85 0)
+    (property "Datasheet" "https://www.onsemi.com/pub/Collateral/NCS210R-D.PDF" (at 101.6 57.15 0)
+      (effects (font (size 1.27 1.27)) hide)
+    )
+    (pin "1")
+    (pin "2")
+    (pin "3")
+    (pin "4")
+    (pin "5")
+    (pin "6")
+    (instances
+      (project "PCBschematic"
+        (path "/cc300af8-7dc6-4303-a7a3-6c9320b23fa8"
+          (reference "U3") (unit 1)
+        )
+        (path "/cc300af8-7dc6-4303-a7a3-6c9320b23fa8/ee85df54-7893-4d17-a059-faa4a0440549"
+          (reference "U2") (unit 1)
+        )
+      )
+    )
+  )
+  (symbol (lib_id "power:GND") (at 101.6 66.04 0) (unit 1)
+    (in_bom yes) (on_board yes) (dnp no) (fields_autoplaced)
+    (property "Reference" "#PWR04" (at 101.6 72.39 0)
+      (effects (font (size 1.27 1.27)) hide)
+    )
+    (property "Value" "GND" (at 101.6 71.12 0)
       (effects (font (size 1.27 1.27)))
     )
-    (property "Footprint" "" (at 91.44 64.77 0)
+    (property "Footprint" "" (at 101.6 66.04 0)
       (effects (font (size 1.27 1.27)) hide)
     )
-    (property "Datasheet" "" (at 91.44 64.77 0)
+    (property "Datasheet" "" (at 101.6 66.04 0)
       (effects (font (size 1.27 1.27)) hide)
     )

Commit message: stm32_pin_parametre
Parts:
- added C5 (x3): 0.1, Capacitor_SMD:C_0603_1608Metric_Pad1.08x0.95mm_HandSolder, symbol Device:C_Small
- added C5: 0.1u, Capacitor_SMD:C_0603_1608Metric_Pad1.08x0.95mm_HandSolder, symbol Device:C_Small
- added D2 (x3): VS-30BQ0115HM3, Diode_SMD:D_0201_0603Metric_Pad0.64x0.40mm_HandSolder, symbol Diode:1N5400
- added J3 (x3): Conn_01x02, Connector_JST:JST_XH_B2B-XH-A_1x02_P2.50mm_Vertical, symbol Connector_Generic:Conn_01x02
- added Q1 (x3): SQ2310ES, Transistor_Power_Module:Littelfuse_Package_H_XBN2MM, symbol Simulation_SPICE:NMOS
- added R1 (x3): R_Small, Resistor_SMD:R_0603_1608Metric_Pad0.98x0.95mm_HandSolder, symbol Device:R_Small
- added U3 (x3): NCS210, Package_TO_SOT_SMD:SOT-363_SC-70-6, symbol Amplifier_Current:NCS210
- D2: footprint Diode_THT:D_DO-201AD_P15.24mm_Horizontal -> Diode_SMD:D_0603_1608Metric_Pad1.05x0.95mm_HandSolder
- J3: footprint (none) -> Connector_JST:JST_XH_B2B-XH-A_1x02_P2.50mm_Vertical
- Q1: footprint (none) -> Transistor_Power_Module:Littelfuse_Package_H_XBN2MM
- R1: footprint (none) -> Resistor_SMD:R_0603_1608Metric_Pad0.98x0.95mm_HandSolder
Connections:
- net GND: now also C5.1, C5.1, C5.1, C5.1, Q1.3 (S), Q1.3 (S), Q1.3 (S), U3.2 (GND), U3.2 (GND), U3.2 (GND)
- net VCC: now also R1.1, R1.1, R1.1, U3.4 (+IN), U3.4 (+IN), U3.4 (+IN)
- net +3.3V: now reaches U3.1 (REF)
- net +3.3V: now also U3.3 (Vs), C5.2, C5.2, C5.2, C5.2, U3.1 (REF), U3.1 (REF), U3.1 (REF), U3.3 (Vs), U3.3 (Vs), U3.3 (Vs)
- net AO1: now reaches U3.6 (OUT)
- new net: D2.1 (K), J3.1 (Pin_1), R1.2, U3.5 (-IN) (x3)
- new net: D2.2 (A), J3.2 (Pin_2), Q1.1 (D) (x3)
- new net AO2: U3.6 (OUT)
- new net AO3: U3.6 (OUT)
- new net AO4: U3.6 (OUT)
- new net PWM_2: Q1.2 (G)
- new net PWM_3: Q1.2 (G)
- new net PWM_4: Q1.2 (G)

Commit message: pcb schematic sans erreur et editeur sans erreur egalement
Parts:
- D2: footprint Diode_SMD:D_0201_0603Metric_Pad0.64x0.40mm_HandSolder -> Diode_SMD:D_0603_1608Metric_Pad1.05x0.95mm_HandSolder
Changed lines of the file:
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@@
   (junction (at 171.45 58.42) (diameter 0) (color 0 0 0 0)
   )
+  (junction (at 171.45 102.87) (diameter 0) (color 0 0 0 0)
+  )
   (junction (at 171.45 111.76) (diameter 0) (color 0 0 0 0)
   )
@@
     (stroke (width 0) (type default))
   )
+  (wire (pts (xy 171.45 102.87) (xy 171.45 104.14))
+    (stroke (width 0) (type default))
+  )
   (wire (pts (xy 68.58 123.19) (xy 59.69 123.19))
     (stroke (width 0) (type default))
@@
     (stroke (width 0) (type default))
   )
-  (wire (pts (xy 171.45 101.6) (xy 171.45 104.14))
+  (wire (pts (xy 171.45 101.6) (xy 171.45 102.87))
     (stroke (width 0) (type default))
   )
@@
       (effects (font (size 1.27 1.27)) (justify left))
     )
-    (property "Footprint" "Diode_SMD:D_0201_0603Metric_Pad0.64x0.40mm_HandSolder" (at 158.115 64.77 0)
+    (property "Footprint" "Diode_SMD:D_0603_1608Metric_Pad1.05x0.95mm_HandSolder" (at 158.115 64.77 0)
       (effects (font (size 1.27 1.27)) hide)
     )
@@
       (effects (font (size 1.27 1.27)) (justify left))
     )
-    (property "Footprint" "Diode_SMD:D_0201_0603Metric_Pad0.64x0.40mm_HandSolder" (at 55.245 119.38 0)
+    (property "Footprint" "Diode_SMD:D_0603_1608Metric_Pad1.05x0.95mm_HandSolder" (at 55.245 119.38 0)
       (effects (font (size 1.27 1.27)) hide)
     )
@@
     )
   )
+  (symbol (lib_id "power:PWR_FLAG") (at 171.45 102.87 270) (unit 1)
+    (in_bom yes) (on_board yes) (dnp no) (fields_autoplaced)
+    (property "Reference" "#FLG02" (at 173.355 102.87 0)
+      (effects (font (size 1.27 1.27)) hide)
+    )
+    (property "Value" "PWR_FLAG" (at 175.26 103.505 90)
+      (effects (font (size 1.27 1.27)) (justify left))
+    )
+    (property "Footprint" "" (at 171.45 102.87 0)
+      (effects (font (size 1.27 1.27)) hide)
+    )
+    (property "Datasheet" "~" (at 171.45 102.87 0)
+      (effects (font (size 1.27 1.27)) hide)
+    )
+    (pin "1")
+    (instances
+      (project "PCBschematic"
+        (path "/cc300af8-7dc6-4303-a7a3-6c9320b23fa8"
+          (reference "#FLG02") (unit 1)
+        )
+        (path "/cc300af8-7dc6-4303-a7a3-6c9320b23fa8/ee85df54-7893-4d17-a059-faa4a0440549"
+          (reference "#FLG03") (unit 1)
+        )
+      )
+    )
+  )
   (symbol (lib_id "power:GND") (at 68.58 87.63 0) (unit 1)
     (in_bom yes) (on_board yes) (dnp no) (fields_autoplaced)
@@
       (effects (font (size 1.27 1.27)) (justify left))
     )
-    (property "Footprint" "Diode_SMD:D_0201_0603Metric_Pad0.64x0.40mm_HandSolder" (at 158.115 115.57 0)
-      (effects (font (size 1.27 1.27)) hide)
-    )
+    (property "Footprint" "Diode_SMD:D_0603_1608Metric_Pad1.05x0.95mm_HandSolder" (at 158.115 115.57 0)
+      (effects (font (size 1.27 1.27)) hide)
+    )
