File: PCBschematic/PCBschematic.kicad_pcb (KiCad board)
At the start: 2 copper layers, 263.8 x 220 mm, 49 parts, among them J3 Conn_01x02, J4 Conn_02x07_Odd_Even, J5 Conn_01x02, J6 Conn_01x02, J7 Conn_01x02, J8 batterie_regulation_centralei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, J9 Conn_01x08, Q1 SQ2310ES, Q2 SQ2310ES, Q3 SQ2310ES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

Commit message: ajout des GND sur le pcb
Parts:
- moved H2 6.86 mm to (374.5, 40.1)
- moved H3 3.16 mm to (127.0, 235.0)
- moved H4 1.00 mm to (375.0, 235.0)
Routing:
- net GND: track 1062.4 -> 1058.2 mm
- net (no net): vias 0 -> 358
Other:
- board size 263.8 x 220 mm -> 264 x 204.6 mm
- board text added: "B"
- board text added: "DRONE"
- board text added: "T"
