File: Hardware/PCBschematic/untitled.kicad_sch (KiCad schematic)
At the start: 24 parts, among them J3 Conn_01x02, Q1 SQ2310ES, U3 NCS210

Commit message: correction
Parts:
- D2: footprint Diode_SMD:D_0603_1608Metric_Pad1.05x0.95mm_HandSolder -> (none)
- Q1: footprint Transistor_Power_Module:Littelfuse_Package_H_XBN2MM -> Package_TO_SOT_SMD:SOT-23
- R1: value R_Small -> 100m
- U3: footprint Package_TO_SOT_SMD:SOT-363_SC-70-6 -> footprints:SC70-6_ONS
Connections:
- net GND: now also U3.1 (REF), U3.1 (REF), U3.1 (REF), U3.1 (REF)
- net +3.3V renamed +3.3VA
- net +3.3VA: no longer U3.1 (REF), U3.1 (REF), U3.1 (REF), U3.1 (REF)

Commit message: pcb en cours de correction
Parts:
- removed R1 (x3): R_Small, Resistor_SMD:R_0603_1608Metric_Pad0.98x0.95mm_HandSolder, symbol Device:R_Small
- removed R1: 100m, Resistor_SMD:R_0603_1608Metric_Pad0.98x0.95mm_HandSolder, symbol Device:R_Small
- added R1, R4, R6, R7: R_Small, Resistor_SMD:R_0603_1608Metric_Pad0.98x0.95mm_HandSolder, symbol Device:R_Small
- C5: value 0.1 -> 0.1u
- D2: footprint (none) -> Diode_SMD:D_SMC_Handsoldering
Connections:
- net VCC: now also R1.1, R4.1, R6.1, R7.1
- net at D2.1 (K), J3.1 (Pin_1), U3.5 (-IN): now also R4.2
- net at D2.1 (K), J3.1 (Pin_1), U3.5 (-IN): now also R7.2
- net at D2.1 (K), J3.1 (Pin_1), U3.5 (-IN): now also R6.2
- net at D2.1 (K), J3.1 (Pin_1), U3.5 (-IN): now also R1.2

Commit message: avancementpcb
Parts:
- D2: footprint Diode_SMD:D_SMC_Handsoldering -> Diode_SMD:D_SMB-SMC_Universal_Handsoldering
Changed lines of the file:
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@@
       (effects (font (size 1.27 1.27)) (justify left))
     )
-    (property "Footprint" "Diode_SMD:D_SMC_Handsoldering" (at 158.115 64.77 0)
+    (property "Footprint" "Diode_SMD:D_SMB-SMC_Universal_Handsoldering" (at 158.115 64.77 0)
       (effects (font (size 1.27 1.27)) hide)
     )
@@
       (effects (font (size 1.27 1.27)) (justify left))
     )
-    (property "Footprint" "Diode_SMD:D_SMC_Handsoldering" (at 55.245 66.04 0)
+    (property "Footprint" "Diode_SMD:D_SMB-SMC_Universal_Handsoldering" (at 55.245 66.04 0)
       (effects (font (size 1.27 1.27)) hide)
     )
@@
       (effects (font (size 1.27 1.27)) (justify left))
     )
-    (property "Footprint" "Diode_SMD:D_SMC_Handsoldering" (at 55.245 119.38 0)
+    (property "Footprint" "Diode_SMD:D_SMB-SMC_Universal_Handsoldering" (at 55.245 119.38 0)
       (effects (font (size 1.27 1.27)) hide)
     )
@@
       (effects (font (size 1.27 1.27)) (justify left))
     )
-    (property "Footprint" "Diode_SMD:D_SMC_Handsoldering" (at 158.115 115.57 0)
-      (effects (font (size 1.27 1.27)) hide)
-    )
+    (property "Footprint" "Diode_SMD:D_SMB-SMC_Universal_Handsoldering" (at 158.115 115.57 0)
+      (effects (font (size 1.27 1.27)) hide)
+    )
