File: Hardware/PCBschematic/_autosave-untitled.kicad_sch (KiCad schematic)
At the start: 24 parts, among them J3 Conn_01x02, Q1 SQ2310ES, U3 NCS210

Commit message: pcbpluspetot
Parts:
- D2: footprint Diode_SMD:D_SMB-SMC_Universal_Handsoldering -> mesempreintes:DiodeVS-30BQ015HM3
Changed lines of the file:
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@@
       (effects (font (size 1.27 1.27)) (justify left))
     )
-    (property "Footprint" "Diode_SMD:D_SMB-SMC_Universal_Handsoldering" (at 158.115 64.77 0)
+    (property "Footprint" "mesempreintes:DiodeVS-30BQ015HM3" (at 158.115 64.77 0)
       (effects (font (size 1.27 1.27)) hide)
     )
@@
       (effects (font (size 1.27 1.27)) (justify left))
     )
-    (property "Footprint" "Diode_SMD:D_SMB-SMC_Universal_Handsoldering" (at 55.245 66.04 0)
+    (property "Footprint" "mesempreintes:DiodeVS-30BQ015HM3" (at 55.245 66.04 0)
       (effects (font (size 1.27 1.27)) hide)
     )
@@
       (effects (font (size 1.27 1.27)) (justify left))
     )
-    (property "Footprint" "Diode_SMD:D_SMB-SMC_Universal_Handsoldering" (at 55.245 119.38 0)
+    (property "Footprint" "mesempreintes:DiodeVS-30BQ015HM3" (at 55.245 119.38 0)
       (effects (font (size 1.27 1.27)) hide)
     )
@@
       (effects (font (size 1.27 1.27)) (justify left))
     )
-    (property "Footprint" "Diode_SMD:D_SMB-SMC_Universal_Handsoldering" (at 158.115 115.57 0)
-      (effects (font (size 1.27 1.27)) hide)
-    )
+    (property "Footprint" "mesempreintes:DiodeVS-30BQ015HM3" (at 158.115 115.57 0)
+      (effects (font (size 1.27 1.27)) hide)
+    )
