File: Hardware/PCBschematic/PCBschematic.kicad_pcb (KiCad board)
At the start: 2 copper layers, 45 parts, among them J3 Conn_01x02, J4 Conn_02x07_Odd_Even, J5 Conn_01x02, J6 Conn_01x02, J7 Conn_01x02, J8 batterie, J9 Conn_01x08, Q1 SQ2310ES, Q2 SQ2310ES, Q3 SQ2310ES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

Commit message: pcb en cours de correction
Parts:
- removed R8: 100m, Resistor_SMD:R_0603_1608Metric_Pad0.98x0.95mm_HandSolder
- added D1: VS-30BQ0115HM3, Diode_SMD:D_SMC_Handsoldering, F.Cu at (89.9, 101.3)
- added D5: VS-30BQ0115HM3, Diode_SMD:D_SMC_Handsoldering, F.Cu at (89.9, 109.0)
- added D6: VS-30BQ0115HM3, Diode_SMD:D_SMC_Handsoldering, F.Cu at (89.9, 116.8)
- added D7: VS-30BQ0115HM3, Diode_SMD:D_SMC_Handsoldering, F.Cu at (89.9, 124.5)
- added R4: R_Small, Resistor_SMD:R_0603_1608Metric_Pad0.98x0.95mm_HandSolder, F.Cu at (178.4, 137.0)
- C10, C7, C9: value 0.1 -> 0.1u
- moved H3 178.0 mm to (192.0, 137.0)
- moved H1 165.3 mm to (192.0, 94.0)
- moved J3 164.2 mm to (197.9, 145.1)
- moved Q1 153.2 mm to (198.9, 140.3), turned to 180 degrees
- moved C7 153.2 mm to (196.3, 137.2), turned to -90 degrees
- moved R6 148.6 mm to (201.7, 137.0), turned to 90 degrees
- moved U2 148.1 mm to (198.9, 137.3)
- moved U6 147.7 mm to (185.9, 108.3)
- moved R1 139.5 mm to (187.6, 136.7), turned to 90 degrees
- moved J7 137.8 mm to (183.7, 144.8)
- moved C10 137.6 mm to (182.1, 136.9), turned to -90 degrees
- moved L1 137.1 mm to (160.0, 120.2), turned to 180 degrees
- moved J5 136.6 mm to (166.1, 145.1)
- moved J6 136.5 mm to (174.6, 145.0)
- moved SW2 135.6 mm to (154.8, 124.7), turned to -90 degrees
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Connections:
- R1 pad 2: Net-(D1-K) -> Net-(D7-K)
- R6 pad 2: Net-(D5-K) -> Net-(D1-K)
- R7 pad 2: Net-(D6-K) -> Net-(D5-K)
Routing:
- net +3.3V: track 0.00 -> 55.7 mm
- net GND: track 0.00 -> 32.1 mm
- net USART2_TX: track 0.00 -> 28.6 mm, vias 0 -> 2
- net USART2_RX: track 0.00 -> 27.8 mm, vias 0 -> 2
- net Net-(D1-K): track 0.00 -> 19.4 mm
- net Net-(D5-K): track 0.00 -> 17.9 mm
- net Net-(D6-K): track 0.00 -> 16.2 mm
- net +7.5V: track 0.00 -> 15.8 mm
- net Net-(D7-K): track 0.00 -> 14.7 mm
- net I2C_SDA: track 0.00 -> 13.1 mm
- net I2C_SCL: track 0.00 -> 12.4 mm
- net SWDCK: track 0.00 -> 10.4 mm
- net +3.3VA: track 0.00 -> 9.97 mm
- net Reset_Buton : track 0.00 -> 8.64 mm
- net SWDIO: track 0.00 -> 7.89 mm
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- added copper zone on B.Cu, net GND
- added copper zone on F.Cu, net GND
Other:
- board outline added: 85 x 65 mm

Commit message: avancementpcb
Parts:
- D1, D5, D6, D7: footprint Diode_SMD:D_SMC_Handsoldering -> Diode_SMD:D_SMB-SMC_Universal_Handsoldering
- moved D6 84.5 mm to (173.2, 102.2), turned to 90 degrees
- moved D1 84.2 mm to (168.2, 132.1), turned to -90 degrees
- moved J7 64.3 mm to (135.7, 102.1), turned to 180 degrees
- moved R1 61.8 mm to (131.8, 110.3), turned to -90 degrees
- moved Q4 60.3 mm to (134.6, 106.8), turned to 0 degrees
- moved D5 58.4 mm to (144.1, 130.8), turned to -90 degrees
- moved U5 56.9 mm to (134.6, 109.9), turned to 180 degrees
- moved D7 56.1 mm to (142.1, 103.9), turned to 90 degrees
- moved C10 52.3 mm to (137.2, 110.0), turned to 90 degrees
- moved J6 45.1 mm to (182.0, 100.5), turned to 180 degrees
- moved Q3 35.6 mm to (180.5, 105.1), turned to 0 degrees
- moved J8 33.1 mm to (186.9, 129.9), turned to 90 degrees
- moved C8 33.0 mm to (133.1, 125.2)
- moved J5 33.0 mm to (135.1, 133.3)
- moved Q2 33.0 mm to (135.8, 128.6)
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Routing:
- net +3.3VA: track 9.97 -> 177.6 mm, vias 0 -> 11
- net GND: track 32.1 -> 162.8 mm, vias 0 -> 14
- net VCC: track 3.69 -> 114.2 mm, vias 0 -> 4
- net PWM_2: track 0.00 -> 104.2 mm, vias 0 -> 8
- net AO1: track 0.00 -> 81.4 mm, vias 0 -> 8
- net AO3: track 0.00 -> 57.1 mm, vias 0 -> 2
- net PWM_1: track 0.00 -> 39.2 mm, vias 0 -> 2
- net PWM_3: track 0.00 -> 31.8 mm, vias 0 -> 2
- net PWM_4: track 0.00 -> 28.6 mm, vias 0 -> 2
- net Net-(D1-K): track 19.4 -> 46.3 mm, vias 0 -> 2
- net AO4: track 0.00 -> 25.7 mm, vias 0 -> 2
- net +3.3V: track 55.7 -> 81.1 mm, vias 0 -> 2
- net Reset_Buton : track 8.64 -> 32.7 mm, vias 0 -> 2
- net Net-(D7-K): track 14.7 -> 26.8 mm, vias 0 -> 2
- net Net-(D1-A): track 4.11 -> 16.2 mm, vias 0 -> 2
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
Commit message: pcb_mise_en_place_okay_reste_3_erreurs git commit -m pcb_mise_en_place_okay_reste_3_erreurs
Parts:
- moved H3 2.92 mm to (188.7, 138.7)
- moved H1 2.58 mm to (188.3, 94.8)
- moved H4 2.38 mm to (127.1, 138.7)
- moved R2 0.71 mm to (150.1, 106.5)
- moved D2 0.61 mm to (150.2, 109.9)
- moved C1 0.37 mm to (143.0, 117.2), turned to 90 degrees
- moved C9 0.36 mm to (183.8, 109.1)
- moved D3 0.24 mm to (152.1, 110.2)
- moved C7 0.23 mm to (172.9, 125.8)
- moved U4 0.20 mm to (181.1, 109.4)
- moved H2 0.10 mm to (127.3, 95.5)
Routing:
- net GND: track 162.8 -> 167.0 mm
- net I2C_SCL: track 23.7 -> 26.5 mm
- net I2C_SDA: track 18.9 -> 21.0 mm
- net PWM_4: track 28.6 -> 29.9 mm
- net +3.3VA: track 177.6 -> 178.3 mm
- net Reset_Buton : track 32.7 -> 33.3 mm
Other:
- board size 85 x 65 mm -> 69.5 x 50.9 mm

Commit message: modif pcb
Routing:
- net GND: track 167.0 -> 202.7 mm, vias 14 -> 18

Commit message: modif pcb
Parts:
- moved H1 1.03 mm to (189.2, 95.3)
- moved H4 0.51 mm to (127.6, 138.6)
- moved H3 0.22 mm to (188.6, 138.9)
Routing:
- net GND: track 202.7 -> 212.4 mm, vias 18 -> 20
- net VCC: track 114.2 -> 115.4 mm

Commit message: routage v1
Parts:
- moved D7 1.70 mm to (142.1, 102.2)
- moved C10 1.60 mm to (136.9, 108.4)
- moved Q4 1.60 mm to (134.3, 105.2)
- moved R1 1.60 mm to (131.4, 108.7)
- moved U5 1.60 mm to (134.3, 108.3)
- moved J7 1.58 mm to (135.7, 100.5)
- moved J5 1.33 mm to (133.8, 133.7)
- moved H3 1.28 mm to (187.8, 137.9)
- moved H2 0.78 mm to (126.7, 95.0)
- moved D5 0.46 mm to (143.8, 130.5)
- moved C8 0.46 mm to (132.8, 124.9)
- moved Q2 0.46 mm to (135.5, 128.3)
- moved R7 0.46 mm to (138.1, 124.9)
- moved U3 0.46 mm to (135.5, 125.2)
Connections:
- R7 pad 1: VCC -> +3.3VA
- U3 pad 4: VCC -> +3.3VA
Routing:
- net VCC: track 115.4 -> 92.8 mm, vias 4 -> 8
- net PWM_2: track 104.2 -> 123.7 mm
- net GND: track 212.4 -> 220.7 mm
- net +3.3VA: track 178.3 -> 185.3 mm
- net AO1: track 81.4 -> 86.6 mm, vias 8 -> 6
- net USART2_RX: track 28.7 -> 27.2 mm
- net PWM_1: track 39.2 -> 40.6 mm
- net AO4: track 25.7 -> 27.1 mm
- net Net-(D5-A): track 11.3 -> 12.7 mm
Other:
- board size 69.5 x 50.9 mm -> 69.6 x 51.1 mm

Commit message: pcbpluspetot
Parts:
- C1, C2, C3, C4, C5, C6, D2, D3, D4, J4, L1, R2, R3, R5, U1, U6: moved to B.Cu
- D1, D5: footprint Diode_SMD:D_SMB-SMC_Universal_Handsoldering -> mesempreintes:DiodeVS-30BQ015HM3; moved to B.Cu
- D6, D7: footprint Diode_SMD:D_SMB-SMC_Universal_Handsoldering -> mesempreintes:DiodeVS-30BQ015HM3
- moved J9 35.5 mm to (145.4, 130.7), turned to 0 degrees
- moved C11 22.1 mm to (152.3, 122.1)
- moved J8 21.5 mm to (169.2, 117.7)
- moved C9 21.2 mm to (162.6, 109.5)
- moved R4 21.2 mm to (157.1, 110.1)
- moved U4 21.2 mm to (159.9, 109.8)
- moved U6 21.2 mm to (168.6, 108.5)
- moved Q3 20.7 mm to (159.8, 106.8)
- moved H1 19.9 mm to (170.2, 101.2)
- moved H3 19.3 mm to (169.4, 132.0)
- moved SW2 18.3 mm to (151.4, 106.7), turned to 90 degrees
- moved J6 18.0 mm to (164.1, 101.8)
- moved R2 18.0 mm to (148.7, 124.4), turned to -90 degrees
- moved R6 18.0 mm to (160.9, 121.7), turned to 180 degrees
- moved R3 16.7 mm to (150.4, 124.4), turned to -90 degrees
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Connections:
- R7 pad 1: +3.3VA -> VCC
- U3 pad 4: +3.3VA -> VCC
Routing:
- net GND: track 220.7 -> 0.00 mm, vias 20 -> 0
- net +3.3VA: track 185.3 -> 0.00 mm, vias 11 -> 0
- net PWM_2: track 123.7 -> 0.00 mm, vias 8 -> 0
- net VCC: track 92.8 -> 0.00 mm, vias 8 -> 0
- net AO1: track 86.6 -> 0.00 mm, vias 6 -> 0
- net +3.3V: track 81.4 -> 0.00 mm, vias 2 -> 0
- net AO3: track 57.2 -> 0.00 mm, vias 2 -> 0
- net Net-(D1-K): track 46.3 -> 0.00 mm, vias 2 -> 0
- net PWM_1: track 40.6 -> 0.00 mm, vias 2 -> 0
- net Reset_Buton : track 33.3 -> 0.00 mm, vias 2 -> 0
- net PWM_3: track 31.8 -> 0.00 mm, vias 2 -> 0
- net PWM_4: track 30.3 -> 0.00 mm, vias 2 -> 0
- net USART2_TX: track 29.7 -> 0.00 mm, vias 2 -> 0
- net Net-(D5-K): track 28.7 -> 0.00 mm, vias 2 -> 0
- net USART2_RX: track 27.2 -> 0.00 mm, vias 2 -> 0
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
Commit message: pcb_tailledrone
Parts:
- C1, C2, C3, C4, C5, C6, D2, D3, D4, J4, L1, R2, R3, R5, U1, U6: moved to F.Cu
- D6, D7: moved to B.Cu
- H1, H2, H3, H4: footprint MountingHole:MountingHole_3.2mm_M3_DIN965_Pad -> MountingHole:MountingHole_2.2mm_M2_DIN965_Pad
- moved L1 129.8 mm to (54.8, 38.4)
- moved C5 126.5 mm to (56.8, 38.5)
- moved D6 125.8 mm to (68.8, 31.8), turned to 0 degrees
- moved J4 124.8 mm to (58.8, 44.8)
- moved C6 123.9 mm to (58.4, 38.5)
- moved C2 121.4 mm to (59.9, 38.5)
- moved J6 121.1 mm to (70.0, 25.5)
- moved Q4 120.7 mm to (53.7, 30.4)
- moved U5 120.7 mm to (53.7, 33.6)
- moved R1 120.6 mm to (51.0, 34.2)
- moved C10 120.4 mm to (56.2, 34.2)
- moved Q3 119.1 mm to (68.5, 30.2)
- moved U4 118.8 mm to (68.7, 33.6)
- moved C4 118.8 mm to (61.5, 38.6)
- moved C9 118.6 mm to (71.2, 33.8)
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Routing:
- net GND: track 0.00 -> 154.4 mm, vias 0 -> 4
- net +3.3V: track 0.00 -> 86.8 mm, vias 0 -> 4
- net +3.3VA: track 0.00 -> 84.0 mm, vias 0 -> 3
- net PWM_3: track 0.00 -> 41.2 mm, vias 0 -> 2
- net AO1: track 0.00 -> 40.3 mm, vias 0 -> 2
- net Reset_Buton : track 0.00 -> 39.9 mm, vias 0 -> 2
- net PWM_4: track 0.00 -> 32.1 mm
- net AO4: track 0.00 -> 31.0 mm, vias 0 -> 2
- net VCC: track 0.00 -> 30.0 mm, vias 0 -> 2
- net I2C_SDA: track 0.00 -> 27.1 mm, vias 0 -> 4
- net PWM_1: track 0.00 -> 24.6 mm, vias 0 -> 2
- net Net-(D7-K): track 0.00 -> 23.7 mm, vias 0 -> 2
- net SWDIO: track 0.00 -> 23.6 mm, vias 0 -> 2
- net I2C_SCL: track 0.00 -> 23.2 mm, vias 0 -> 2
- net Net-(D5-K): track 0.00 -> 22.2 mm, vias 0 -> 2
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- removed copper zone on B.Cu, net GND
- removed copper zone on F.Cu, net GND
Other:
- board size 69.6 x 51.1 mm -> 32 x 80 mm
