File: Hardware/PCBschematic/PCBschematic.kicad_pcb (KiCad board)
At the start: 2 copper layers, 32 x 80 mm, 49 parts, among them J3 Conn_01x02, J4 Conn_02x07_Odd_Even, J5 Conn_01x02, J6 Conn_01x02, J7 Conn_01x02, J8 batterie, J9 Conn_01x08, Q1 SQ2310ES, Q2 SQ2310ES, Q3 SQ2310ES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

Commit message: nouveau pcb
Routing:
- net VCC: track 30.0 -> 131.2 mm, vias 2 -> 5
- net AO2: track 0.00 -> 59.6 mm, vias 0 -> 4
- net PWM_2: track 0.00 -> 58.1 mm, vias 0 -> 2
- net Start_Buton: track 0.00 -> 27.7 mm, vias 0 -> 2
- net USART2_RX: track 0.00 -> 24.0 mm, vias 0 -> 3
- net AO3: track 0.00 -> 22.2 mm, vias 0 -> 2
- net USART2_TX: track 0.00 -> 20.0 mm, vias 0 -> 2
- net Reset_Buton : track 39.9 -> 49.2 mm
- net +3.3V: track 86.8 -> 94.2 mm
- net SWDIO: track 23.6 -> 29.9 mm
- net PWM_4: track 32.1 -> 34.6 mm
- net GND: track 154.4 -> 152.1 mm
- net AO4: track 31.0 -> 28.8 mm
- net Net-(D6-K): track 19.6 -> 21.4 mm
- net PWM_1: track 24.6 -> 23.4 mm, vias 2 -> 1
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
Commit message: routage v2
Parts:
- moved C11 1.52 mm to (70.8, 65.8)
- moved R6 0.11 mm to (72.0, 88.4)
Routing:
- net GND: track 152.1 -> 256.8 mm, vias 4 -> 10
- net PWM_1: track 23.4 -> 78.4 mm, vias 1 -> 4
- net +3.3VA: track 84.0 -> 128.6 mm, vias 3 -> 6
- net SWDCK: track 0.00 -> 36.2 mm, vias 0 -> 2
- net Net-(D1-K): track 2.48 -> 26.2 mm, vias 0 -> 2
- net Net-(D6-A): track 3.80 -> 11.1 mm, vias 0 -> 1
- net Net-(D7-A): track 4.18 -> 10.9 mm, vias 0 -> 1
- net +3.3V: track 94.2 -> 87.9 mm
- net Net-(D5-K): track 22.2 -> 28.3 mm, vias 2 -> 3
- net Net-(D5-A): track 4.08 -> 9.46 mm, vias 0 -> 1
- net Net-(D1-A): track 4.25 -> 9.32 mm, vias 0 -> 1
- net Net-(D6-K): track 21.4 -> 25.3 mm, vias 0 -> 1
- net AO1: track 40.5 -> 43.7 mm
- net Net-(D7-K): track 24.6 -> 27.6 mm, vias 2 -> 3
- net AO2: track 59.6 -> 61.6 mm
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- added copper zone on B.Cu, net GND
- added copper zone on F.Cu, net GND

Commit message: v2_nom
Other:
- board text added: "Drone_1A"
Changed lines of the file:
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@@
   (gr_arc locked (start 77.25 96.25) (mid 75.785534 99.785534) (end 72.25 101.25)
     (stroke (width 0.1) (type default)) (layer "Edge.Cuts"))
+  (gr_text "Drone_1A\n" (at 47.75 41.5 90) (layer "F.Cu")
+    (effects (font (size 1.5 1.5) (thickness 0.3) bold) (justify left bottom))
+  )
+  (gr_text "Drone_1A\n\n" (at 50.25 31.25 90) (layer "B.Cu")
+    (effects (font (size 1.5 1.5) (thickness 0.3) bold) (justify left bottom mirror))
+  )
   (segment (start 75.34 44.54) (end 74.46 44.54) (width 0.3) (layer "F.Cu") (net 1))
   (segment (start 60.898629 51.28) (end 59.455 51.28) (width 0.3) (layer "F.Cu") (net 1))
@@
   (via (at 58 34.75) (size 0.8) (drill 0.6) (layers "F.Cu" "B.Cu") (net 4))
   (segment (start 46.5 89.369336) (end 49.565332 92.434668) (width 0.5) (layer "B.Cu") (net 4))
-  (segment (start 74.5 34.5) (end 74.5 32.5) (width 0.5) (layer "B.Cu") (net 4))
-  (segment (start 74.5 34.75) (end 74.5 34.5) (width 0.5) (layer "B.Cu") (net 4))
-  (segment (start 74.5 32.5) (end 74.25 32.25) (width 0.5) (layer "B.Cu") (net 4))
-  (segment (start 65.5 36.25) (end 66 35.75) (width 0.5) (layer "B.Cu") (net 4))
+  (segment (start 74.25 32.25) (end 73.75 32.25) (width 0.5) (layer "B.Cu") (net 4))
   (segment (start 58 34.75) (end 58 35.5) (width 0.3) (layer "B.Cu") (net 4))
+  (segment (start 73.5 35.75) (end 74.5 34.75) (width 0.5) (layer "B.Cu") (net 4))
   (segment (start 52.75 39.5) (end 53 39.75) (width 0.3) (layer "B.Cu") (net 4))
   (segment (start 64.75 90.25) (end 60.85 94.15) (width 0.5) (layer "B.Cu") (net 4))
@@
   (segment (start 53.75 36.25) (end 52.75 37.25) (width 0.3) (layer "B.Cu") (net 4))
   (segment (start 52.75 37.25) (end 52.75 39.5) (width 0.3) (layer "B.Cu") (net 4))
+  (segment (start 66 35.75) (end 73.5 35.75) (width 0.5) (layer "B.Cu") (net 4))
+  (segment (start 65.5 36.25) (end 66 35.75) (width 0.5) (layer "B.Cu") (net 4))
   (segment (start 57.25 36.25) (end 53.75 36.25) (width 0.3) (layer "B.Cu") (net 4))
   (segment (start 58 35.5) (end 57.25 36.25) (width 0.3) (layer "B.Cu") (net 4))
-  (segment (start 73.5 35.75) (end 74.5 34.75) (width 0.5) (layer "B.Cu") (net 4))
-  (segment (start 66 35.75) (end 73.5 35.75) (width 0.5) (layer "B.Cu") (net 4))
+  (segment (start 74.5 34.75) (end 74.5 32.5) (width 0.5) (layer "B.Cu") (net 4))
   (segment (start 53.25 39.75) (end 46.5 46.5) (width 0.5) (layer "B.Cu") (net 4))
-  (segment (start 73.75 32.25) (end 74.25 32.25) (width 0.5) (layer "B.Cu") (net 4))
+  (segment (start 74.5 32.5) (end 74.25 32.25) (width 0.5) (layer "B.Cu") (net 4))
   (segment (start 72.75 62.3) (end 75.95 65.5) (width 0.5) (layer "F.Cu") (net 5))
   (segment (start 72.75 58) (end 72.75 62.3) (width 0.5) (layer "F.Cu") (net 5))
@@
   (segment (start 57.055556 29.944444) (end 57.055556 30.614444) (width 0.3) (layer "B.Cu") (net 28))
   (segment (start 57.055556 30.614444) (end 55.97 31.7) (width 0.3) (layer "B.Cu") (net 28))
+  (segment (start 57 81.975) (end 57 78.25) (width 0.3) (layer "F.Cu") (net 29))
   (segment (start 57 78.25) (end 57.25 78) (width 0.3) (layer "F.Cu") (net 29))
-  (segment (start 57 81.975) (end 57 78.25) (width 0.3) (layer "F.Cu") (net 29))
   (segment (start 62 62.075) (end 62.15 61.925) (width 0.3) (layer "F.Cu") (net 29))
   (segment (start 62 64) (end 62 62.075) (width 0.3) (layer "F.Cu") (net 29))

Commit message: routage_V2_fini
Parts:
- C11: value 220uF -> 10uF; footprint Capacitor_SMD:CP_Elec_8x10.5 -> Capacitor_SMD:C_0603_1608Metric_Pad1.08x0.95mm_HandSolder
- SW1, SW2: footprint Button_Switch_THT:SW_Push_1P2T_Vertical_E-Switch_800UDP8P1A1M6 -> Button_Switch_SMD:SW_DIP_SPSTx01_Slide_Copal_CHS-01A_W5.08mm_P1.27mm_JPin
- moved C11 7.24 mm to (65.6, 70.8)
- moved SW1 4.80 mm to (71.4, 41.8)
- moved SW2 3.91 mm to (51.1, 63.7), turned to 180 degrees
- moved R1 0.30 mm to (50.7, 34.2)
Routing:
- net GND: track 256.8 -> 6.70 mm, vias 10 -> 78
- net Reset_Buton : track 48.8 -> 39.9 mm
- net PWM_3: track 41.7 -> 49.6 mm
- net Start_Buton: track 26.9 -> 19.1 mm
- net PWM_1: track 78.4 -> 71.0 mm
- net VCC: track 130.6 -> 124.0 mm
- net AO2: track 61.6 -> 56.9 mm, vias 4 -> 2
- net PWM_4: track 35.2 -> 39.6 mm, vias 0 -> 2
- net AO1: track 43.7 -> 39.8 mm
- net PWM_2: track 58.5 -> 54.9 mm
- net +3.3V: track 87.9 -> 90.4 mm, vias 4 -> 2
- net SWDIO: track 29.3 -> 27.0 mm, vias 2 -> 4
- net Net-(D7-K): track 27.6 -> 25.4 mm, vias 3 -> 1
- net +7.5V: track 22.0 -> 20.3 mm
- net Net-(D6-K): track 25.3 -> 27.0 mm
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