File: Hardware/PCBschematic/PCBschematic.kicad_sch (KiCad schematic)
At the start: 25 parts, among them J4 Conn_02x07_Odd_Even, J8 batterie_regulation_centralei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, J9 Conn_01x08, SW1 SW_Push, SW2 SW_Push, U1 STM32L412KBTx, U6 regulator_17395xx36

Commit message: correction
Parts:
- removed C11: 200u, Capacitor_SMD:C_0603_1608Metric_Pad1.08x0.95mm_HandSolder, symbol Device:C_Small
- added C11: 220uF, Capacitor_SMD:CP_Elec_8x10.5, symbol Device:C_Polarized_Small
- J4: footprint Connector_Molex:Molex_Micro-Fit_3.0_43045-1612_2x08_P3.00mm_Vertical -> Connector_PinHeader_1.27mm:PinHeader_2x07_P1.27mm_Vertical_SMD
- J8: value batterie_regulation_centraleinertielle -> batterie
Connections:
- net +7.5V: now also C11.1
- net GND: now also C11.2
Changed lines of the file:
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@@
+    (stroke (width 0) (type default))
+  )
+  (wire (pts (xy 73.66 123.19) (xy 71.12 123.19))
     (stroke (width 0) (type default))
   )
@@
     (stroke (width 0) (type default))
   )
+  (wire (pts (xy 167.64 125.73) (xy 166.37 125.73))
+    (stroke (width 0) (type default))
+  )
   (polyline (pts (xy 123.19 57.15) (xy 123.19 15.24))
     (stroke (width 0) (type default))
@@
     (stroke (width 0) (type default))
   )
-  (wire (pts (xy 168.91 128.27) (xy 166.37 128.27))
+  (wire (pts (xy 167.64 128.27) (xy 166.37 128.27))
     (stroke (width 0) (type default))
   )
@@
     )
   )
-  (global_label "SWDCK" (shape input) (at 168.91 128.27 0) (fields_autoplaced)
-    (effects (font (size 1.27 1.27)) (justify left))
-    (property "Intersheetrefs" "${INTERSHEET_REFS}" (at 178.2867 128.27 0)
+  (global_label "SWDCK" (shape input) (at 167.64 128.27 0) (fields_autoplaced)
+    (effects (font (size 1.27 1.27)) (justify left))
+    (property "Intersheetrefs" "${INTERSHEET_REFS}" (at 177.0167 128.27 0)
       (effects (font (size 1.27 1.27)) (justify left) hide)
     )
@@
     )
   )
-  (global_label "SWDIO" (shape input) (at 166.37 125.73 0) (fields_autoplaced)
-    (effects (font (size 1.27 1.27)) (justify left))
-    (property "Intersheetrefs" "${INTERSHEET_REFS}" (at 175.142 125.73 0)
+  (global_label "SWDIO" (shape input) (at 167.64 125.73 0) (fields_autoplaced)
+    (effects (font (size 1.27 1.27)) (justify left))
+    (property "Intersheetrefs" "${INTERSHEET_REFS}" (at 176.412 125.73 0)
       (effects (font (size 1.27 1.27)) (justify left) hide)
     )
@@
     )
   )
-  (global_label "SWDIO" (shape input) (at 71.12 123.19 0) (fields_autoplaced)
-    (effects (font (size 1.27 1.27)) (justify left))
-    (property "Intersheetrefs" "${INTERSHEET_REFS}" (at 79.892 123.19 0)
+  (global_label "SWDIO" (shape input) (at 73.66 123.19 0) (fields_autoplaced)
+    (effects (font (size 1.27 1.27)) (justify left))
+    (property "Intersheetrefs" "${INTERSHEET_REFS}" (at 82.432 123.19 0)
       (effects (font (size 1.27 1.27)) (justify left) hide)
     )
@@
       (effects (font (size 1.27 1.27)))
     )
-    (property "Footprint" "Connector_Molex:Molex_Micro-Fit_3.0_43045-1612_2x08_P3.00mm_Vertical" (at 158.75 130.81 0)
+    (property "Footprint" "Connector_PinHeader_1.27mm:PinHeader_2x07_P1.27mm_Vertical_SMD" (at 158.75 130.81 0)
       (effects (font (size 1.27 1.27)) hide)
     )
@@
         (path "/cc300af8-7dc6-4303-a7a3-6c9320b23fa8"
           (reference "#PWR05") (unit 1)
+        )
+      )
+    )
+  )
+  (symbol (lib_id "Device:C_Polarized_Small") (at 167.64 81.28 0) (unit 1)
+    (in_bom yes) (on_board yes) (dnp no) (fields_autoplaced)
+    (property "Reference" "C11" (at 170.18 80.0989 0)
+      (effects (font (size 1.27 1.27)) (justify left))
+    )
+    (property "Value" "220uF" (at 170.18 82.6389 0)
+      (effects (font (size 1.27 1.27)) (justify left))
+    )
+    (property "Footprint" "Capacitor_SMD:CP_Elec_8x10.5" (at 167.64 81.28 0)
+      (effects (font (size 1.27 1.27)) hide)
+    )
+    (property "Datasheet" "~" (at 167.64 81.28 0)
+      (effects (font (size 1.27 1.27)) hide)
+    )
+    (pin "1")
+    (pin "2")
+    (instances
+      (project "PCBschematic"
+        (path "/cc300af8-7dc6-4303-a7a3-6c9320b23fa8"
+          (reference "C11") (unit 1)
         )
       )
@@
       (effects (font (size 1.27 1.27)))
     )
-    (property "Value" "batterie_regulation_centraleinertielle" (at 152.4 85.09 0)
+    (property "Value" "batterie" (at 152.4 85.09 0)
       (effects (font (size 1.27 1.27)))
     )
@@
         )
       )
-    )
-  )
-  (symbol (lib_id "Device:C_Small") (at 167.64 81.28 0) (unit 1)
-    (in_bom yes) (on_board yes) (dnp no) (fields_autoplaced)
-    (property "Reference" "C11" (at 170.18 80.6513 0)
-      (effects (font (size 1.27 1.27)) (justify left))
-    )
-    (property "Value" "200u" (at 170.18 83.1913 0)
-      (effects (font (size 1.27 1.27)) (justify left))
-    )
-    (property "Footprint" "Capacitor_SMD:C_0603_1608Metric_Pad1.08x0.95mm_HandSolder" (at 167.64 81.28 0)
-      (effects (font (size 1.27 1.27)) hide)
-    )
-    (property "Datasheet" "~" (at 167.64 81.28 0)
-      (effects (font (size 1.27 1.27)) hide)
-    )
-    (pin "1")
-    (pin "2")
-    (instances
-      (project "PCBschematic"
-        (path "/cc300af8-7dc6-4303-a7a3-6c9320b23fa8"
-          (reference "C11") (unit 1)
-        )
-      )

Commit message: pcb en cours de correction
Other:
- moved on the sheet: C5, C6, L1

Commit message: pcb_tailledrone
Parts:
- H1, H2, H3, H4: footprint MountingHole:MountingHole_3.2mm_M3_DIN965_Pad -> MountingHole:MountingHole_2.2mm_M2_DIN965_Pad
Changed lines of the file:
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@@
       (effects (font (size 1.27 1.27)) (justify left))
     )
-    (property "Footprint" "MountingHole:MountingHole_3.2mm_M3_DIN965_Pad" (at 257.81 27.94 0)
+    (property "Footprint" "MountingHole:MountingHole_2.2mm_M2_DIN965_Pad" (at 257.81 27.94 0)
       (effects (font (size 1.27 1.27)) hide)
     )
@@
       (effects (font (size 1.27 1.27)) (justify left))
     )
-    (property "Footprint" "MountingHole:MountingHole_3.2mm_M3_DIN965_Pad" (at 257.81 38.1 0)
+    (property "Footprint" "MountingHole:MountingHole_2.2mm_M2_DIN965_Pad" (at 257.81 38.1 0)
       (effects (font (size 1.27 1.27)) hide)
     )
@@
       (effects (font (size 1.27 1.27)) (justify left))
     )
-    (property "Footprint" "MountingHole:MountingHole_3.2mm_M3_DIN965_Pad" (at 257.81 22.86 0)
+    (property "Footprint" "MountingHole:MountingHole_2.2mm_M2_DIN965_Pad" (at 257.81 22.86 0)
       (effects (font (size 1.27 1.27)) hide)
     )
@@
       (effects (font (size 1.27 1.27)) (justify left))
     )
-    (property "Footprint" "MountingHole:MountingHole_3.2mm_M3_DIN965_Pad" (at 257.81 33.02 0)
+    (property "Footprint" "MountingHole:MountingHole_2.2mm_M2_DIN965_Pad" (at 257.81 33.02 0)
       (effects (font (size 1.27 1.27)) hide)
     )

Commit message: routage_V2_fini
Parts:
- C11: value 220uF -> 10uF; footprint Capacitor_SMD:CP_Elec_8x10.5 -> Capacitor_SMD:C_0603_1608Metric_Pad1.08x0.95mm_HandSolder
- SW1, SW2: footprint Button_Switch_THT:SW_Push_1P2T_Vertical_E-Switch_800UDP8P1A1M6 -> Button_Switch_SMD:SW_DIP_SPSTx01_Slide_Copal_CHS-01A_W5.08mm_P1.27mm_JPin
Changed lines of the file:
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@@
       (effects (font (size 1.27 1.27)) (justify left))
     )
-    (property "Value" "220uF" (at 170.18 82.6389 0)
-      (effects (font (size 1.27 1.27)) (justify left))
-    )
-    (property "Footprint" "Capacitor_SMD:CP_Elec_8x10.5" (at 167.64 81.28 0)
+    (property "Value" "10uF" (at 170.18 82.6389 0)
+      (effects (font (size 1.27 1.27)) (justify left))
+    )
+    (property "Footprint" "Capacitor_SMD:C_0603_1608Metric_Pad1.08x0.95mm_HandSolder" (at 167.64 81.28 0)
       (effects (font (size 1.27 1.27)) hide)
     )
@@
       (effects (font (size 1.27 1.27)))
     )
-    (property "Footprint" "Button_Switch_THT:SW_Push_1P2T_Vertical_E-Switch_800UDP8P1A1M6" (at 52.07 27.94 0)
+    (property "Footprint" "Button_Switch_SMD:SW_DIP_SPSTx01_Slide_Copal_CHS-01A_W5.08mm_P1.27mm_JPin" (at 52.07 27.94 0)
       (effects (font (size 1.27 1.27)) hide)
     )
@@
       (effects (font (size 1.27 1.27)))
     )
-    (property "Footprint" "Button_Switch_THT:SW_Push_1P2T_Vertical_E-Switch_800UDP8P1A1M6" (at 83.82 27.94 0)
-      (effects (font (size 1.27 1.27)) hide)
-    )
+    (property "Footprint" "Button_Switch_SMD:SW_DIP_SPSTx01_Slide_Copal_CHS-01A_W5.08mm_P1.27mm_JPin" (at 83.82 27.94 0)
+      (effects (font (size 1.27 1.27)) hide)
+    )
