File: Hardware/PCBschematic_20230519/PCBschematic.kicad_sch (KiCad schematic)
At the start: 29 parts, among them J4 Conn_02x07_Odd_Even, J8 batterie, J9 Conn_01x08, SW1 SW_Push, SW2 SW_Push, U1 STM32L412KBTx, U6 regulator_17395xx36

Commit message: ajout description composants sur schématique
Other:
- note added: "Regulator 17395xx36 Maximum Input 36V / 500mA Fixed Output 3.3V, 5V, 12V or 15V"
- note added: "STM32L412xx 1.71 V to 3.6 V power supply 12x communication interfaces"
- note removed: "Regulator"
- note removed: "STM32"
- moved on the sheet: C2, C3, C4
Changed lines of the file:
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@@
   (junction (at 107.95 77.47) (diameter 0) (color 0 0 0 0)
   )
-  (junction (at 53.34 71.12) (diameter 0) (color 0 0 0 0)
+  (junction (at 59.69 72.39) (diameter 0) (color 0 0 0 0)
   )
   (junction (at 185.42 86.36) (diameter 0) (color 0 0 0 0)
@@
   (junction (at 107.95 78.74) (diameter 0) (color 0 0 0 0)
   )
-  (junction (at 53.34 77.47) (diameter 0) (color 0 0 0 0)
-  )
-  (junction (at 41.91 77.47) (diameter 0) (color 0 0 0 0)
+  (junction (at 59.69 78.74) (diameter 0) (color 0 0 0 0)
   )
   (junction (at 167.64 77.47) (diameter 0) (color 0 0 0 0)
   )
+  (junction (at 48.26 78.74) (diameter 0) (color 0 0 0 0)
+  )
   (junction (at 185.42 85.09) (diameter 0) (color 0 0 0 0)
   )
@@
   (junction (at 167.64 76.2) (diameter 0) (color 0 0 0 0)
   )
-  (junction (at 41.91 71.12) (diameter 0) (color 0 0 0 0)
+  (junction (at 48.26 72.39) (diameter 0) (color 0 0 0 0)
   )
   (junction (at 96.52 90.17) (diameter 0) (color 0 0 0 0)
@@
     (stroke (width 0) (type default))
   )
-  (wire (pts (xy 41.91 77.47) (xy 53.34 77.47))
-    (stroke (width 0) (type default))
-  )
-  (wire (pts (xy 53.34 77.47) (xy 63.5 77.47))
+  (wire (pts (xy 48.26 78.74) (xy 59.69 78.74))
+    (stroke (width 0) (type default))
+  )
+  (wire (pts (xy 59.69 78.74) (xy 69.85 78.74))
     (stroke (width 0) (type default))
   )
@@
     (stroke (width 0) (type default))
   )
-  (wire (pts (xy 63.5 72.39) (xy 63.5 71.12))
+  (wire (pts (xy 69.85 73.66) (xy 69.85 72.39))
+    (stroke (width 0) (type default))
+  )
+  (wire (pts (xy 48.26 78.74) (xy 48.26 80.01))
     (stroke (width 0) (type default))
   )
@@
     (stroke (width 0) (type default))
   )
-  (wire (pts (xy 41.91 72.39) (xy 41.91 71.12))
+  (wire (pts (xy 48.26 73.66) (xy 48.26 72.39))
     (stroke (width 0) (type default))
   )
@@
     (stroke (width 0) (type default))
   )
-  (wire (pts (xy 63.5 71.12) (xy 53.34 71.12))
+  (wire (pts (xy 69.85 72.39) (xy 59.69 72.39))
     (stroke (width 0) (type default))
   )
@@
     (stroke (width 0) (type default))
   )
-  (wire (pts (xy 53.34 71.12) (xy 53.34 72.39))
+  (wire (pts (xy 59.69 72.39) (xy 59.69 73.66))
     (stroke (width 0) (type default))
   )
@@
     (stroke (width 0) (type default))
   )
-  (wire (pts (xy 41.91 71.12) (xy 53.34 71.12))
+  (wire (pts (xy 48.26 72.39) (xy 59.69 72.39))
     (stroke (width 0) (type default))
   )
@@
     (effects (font (size 1.27 1.27)) (justify left bottom))
   )
-  (text "STM32" (at 17.78 66.04 0)
+  (text "STM32L412xx\n1.71 V to 3.6 V power supply\n12x communication interfaces"
+    (at 17.78 71.12 0)
     (effects (font (size 1.27 1.27) (thickness 0.254) bold) (justify left bottom))
   )
@@
     (effects (font (size 1.27 1.27)) (justify left bottom))
   )
-  (text "Regulator\n" (at 135.89 66.04 0)
+  (text "Regulator 17395xx36\nMaximum Input 36V / 500mA \nFixed Output 3.3V, 5V, 12V or 15V"
+    (at 135.89 69.85 0)
     (effects (font (size 1.27 1.27)) (justify left bottom))
   )
@@
   )
   (symbol (lib_id "power:+3.3V") (at 55.88 82.55 0) (unit 1)
-    (in_bom yes) (on_board yes) (dnp no) (fields_autoplaced)
+    (in_bom yes) (on_board yes) (dnp no)
     (property "Reference" "#PWR05" (at 55.88 86.36 0)
       (effects (font (size 1.27 1.27)) hide)
     )
-    (property "Value" "+3.3V" (at 55.88 78.74 0)
+    (property "Value" "+3.3V" (at 55.88 80.01 0)
       (effects (font (size 1.27 1.27)))
     )
@@
     )
   )
-  (symbol (lib_id "Device:C_Small") (at 41.91 74.93 0) (unit 1)
-    (in_bom yes) (on_board yes) (dnp no) (fields_autoplaced)
-    (property "Reference" "C2" (at 44.45 74.3013 0)
-      (effects (font (size 1.27 1.27)) (justify left))
-    )
-    (property "Value" "4.7uF" (at 44.45 76.8413 0)
-      (effects (font (size 1.27 1.27)) (justify left))
-    )
-    (property "Footprint" "Capacitor_SMD:C_0603_1608Metric_Pad1.08x0.95mm_HandSolder" (at 41.91 74.93 0)
-      (effects (font (size 1.27 1.27)) hide)
-    )
-    (property "Datasheet" "~" (at 41.91 74.93 0)
+  (symbol (lib_id "Device:C_Small") (at 48.26 76.2 0) (unit 1)
+    (in_bom yes) (on_board yes) (dnp no) (fields_autoplaced)
+    (property "Reference" "C2" (at 50.8 75.5713 0)
+      (effects (font (size 1.27 1.27)) (justify left))
+    )
+    (property "Value" "4.7uF" (at 50.8 78.1113 0)
+      (effects (font (size 1.27 1.27)) (justify left))
+    )
+    (property "Footprint" "Capacitor_SMD:C_0603_1608Metric_Pad1.08x0.95mm_HandSolder" (at 48.26 76.2 0)
+      (effects (font (size 1.27 1.27)) hide)
+    )
+    (property "Datasheet" "~" (at 48.26 76.2 0)
       (effects (font (size 1.27 1.27)) hide)
     )
@@
     )
   )
-  (symbol (lib_id "Device:C_Small") (at 53.34 74.93 0) (unit 1)
-    (in_bom yes) (on_board yes) (dnp no) (fields_autoplaced)
-    (property "Reference" "C3" (at 55.88 74.3013 0)
-      (effects (font (size 1.27 1.27)) (justify left))
-    )
-    (property "Value" "100n" (at 55.88 76.8413 0)
-      (effects (font (size 1.27 1.27)) (justify left))
-    )
-    (property "Footprint" "Capacitor_SMD:C_0603_1608Metric_Pad1.08x0.95mm_HandSolder" (at 53.34 74.93 0)
-      (effects (font (size 1.27 1.27)) hide)
-    )
-    (property "Datasheet" "~" (at 53.34 74.93 0)
+  (symbol (lib_id "Device:C_Small") (at 59.69 76.2 0) (unit 1)
+    (in_bom yes) (on_board yes) (dnp no) (fields_autoplaced)
+    (property "Reference" "C3" (at 62.23 75.5713 0)
+      (effects (font (size 1.27 1.27)) (justify left))
+    )
+    (property "Value" "100n" (at 62.23 78.1113 0)
+      (effects (font (size 1.27 1.27)) (justify left))
+    )
+    (property "Footprint" "Capacitor_SMD:C_0603_1608Metric_Pad1.08x0.95mm_HandSolder" (at 59.69 76.2 0)
+      (effects (font (size 1.27 1.27)) hide)
+    )
+    (property "Datasheet" "~" (at 59.69 76.2 0)
       (effects (font (size 1.27 1.27)) hide)
     )
@@
   )
   (symbol (lib_id "power:+3.3VA") (at 60.96 82.55 0) (unit 1)
-    (in_bom yes) (on_board yes) (dnp no) (fields_autoplaced)
+    (in_bom yes) (on_board yes) (dnp no)
     (property "Reference" "#PWR047" (at 60.96 86.36 0)
       (effects (font (size 1.27 1.27)) hide)
     )
-    (property "Value" "+3.3VA" (at 60.96 78.74 0)
+    (property "Value" "+3.3VA" (at 62.23 80.01 0)
       (effects (font (size 1.27 1.27)))
     )
@@
     )
   )
-  (symbol (lib_id "Device:C_Small") (at 63.5 74.93 0) (unit 1)
-    (in_bom yes) (on_board yes) (dnp no) (fields_autoplaced)
-    (property "Reference" "C4" (at 66.04 74.3013 0)
-      (effects (font (size 1.27 1.27)) (justify left))
-    )
-    (property "Value" "100n" (at 66.04 76.8413 0)
-      (effects (font (size 1.27 1.27)) (justify left))
-    )
-    (property "Footprint" "Capacitor_SMD:C_0603_1608Metric_Pad1.08x0.95mm_HandSolder" (at 63.5 74.93 0)
-      (effects (font (size 1.27 1.27)) hide)
-    )
-    (property "Datasheet" "~" (at 63.5 74.93 0)
+  (symbol (lib_id "Device:C_Small") (at 69.85 76.2 0) (unit 1)
+    (in_bom yes) (on_board yes) (dnp no) (fields_autoplaced)
+    (property "Reference" "C4" (at 72.39 75.5713 0)
+      (effects (font (size 1.27 1.27)) (justify left))
+    )
+    (property "Value" "100n" (at 72.39 78.1113 0)
+      (effects (font (size 1.27 1.27)) (justify left))
+    )
+    (property "Footprint" "Capacitor_SMD:C_0603_1608Metric_Pad1.08x0.95mm_HandSolder" (at 69.85 76.2 0)
+      (effects (font (size 1.27 1.27)) hide)
+    )
+    (property "Datasheet" "~" (at 69.85 76.2 0)
       (effects (font (size 1.27 1.27)) hide)
     )
@@
     )
   )
-  (symbol (lib_id "power:+3.3V") (at 41.91 71.12 0) (unit 1)
-    (in_bom yes) (on_board yes) (dnp no) (fields_autoplaced)
-    (property "Reference" "#PWR015" (at 41.91 74.93 0)
-      (effects (font (size 1.27 1.27)) hide)
-    )
-    (property "Value" "+3.3V" (at 41.91 67.31 0)
-      (effects (font (size 1.27 1.27)))
-    )
-    (property "Footprint" "" (at 41.91 71.12 0)
-      (effects (font (size 1.27 1.27)) hide)
-    )
-    (property "Datasheet" "" (at 41.91 71.12 0)
+  (symbol (lib_id "power:+3.3V") (at 48.26 72.39 0) (unit 1)
+    (in_bom yes) (on_board yes) (dnp no) (fields_autoplaced)
+    (property "Reference" "#PWR015" (at 48.26 76.2 0)
+      (effects (font (size 1.27 1.27)) hide)
+    )
+    (property "Value" "+3.3V" (at 48.26 68.58 0)
+      (effects (font (size 1.27 1.27)))
+    )
+    (property "Footprint" "" (at 48.26 72.39 0)
+      (effects (font (size 1.27 1.27)) hide)
+    )
+    (property "Datasheet" "" (at 48.26 72.39 0)
       (effects (font (size 1.27 1.27)) hide)
     )
@@
     )
   )
-  (symbol (lib_id "power:GND") (at 41.91 77.47 0) (unit 1)
-    (in_bom yes) (on_board yes) (dnp no) (fields_autoplaced)
-    (property "Reference" "#PWR014" (at 41.91 83.82 0)
-      (effects (font (size 1.27 1.27)) hide)
-    )
-    (property "Value" "GND" (at 41.91 82.55 0)
-      (effects (font (size 1.27 1.27)))
-    )
-    (property "Footprint" "" (at 41.91 77.47 0)
-      (effects (font (size 1.27 1.27)) hide)
-    )
-    (property "Datasheet" "" (at 41.91 77.47 0)
-      (effects (font (size 1.27 1.27)) hide)
-    )
+  (symbol (lib_id "power:GND") (at 48.26 80.01 0) (unit 1)
+    (in_bom yes) (on_board yes) (dnp no) (fields_autoplaced)
+    (property "Reference" "#PWR014" (at 48.26 86.36 0)
+      (effects (font (size 1.27 1.27)) hide)
+    )
+    (property "Value" "GND" (at 48.26 85.09 0)
+      (effects (font (size 1.27 1.27)))
+    )
+    (property "Footprint" "" (at 48.26 80.01 0)
+      (effects (font (size 1.27 1.27)) hide)
+    )
+    (property "Datasheet" "" (at 48.26 80.01 0)
+      (effects (font (size 1.27 1.27)) hide)
+    )
